Commit message: ARM control urdf

File: ARM_control/models/robot.urdf (robot description, URDF)
Before this commit: robot petri_arm_placeholder, 8 links, 7 joints
Links:
- removed link link_0
- removed link tool
- added link tool0
Joints:
- removed joint joint_0
- removed joint tool_fixed
- added joint tool0_fixed: type fixed, parent link_5, child tool0, origin xyz=0 0 0 rpy=0 0 0
- joint joint_1: limit lower=0 upper=3.141592653589793 effort=1 velocity=1 -> lower=-3.14159 upper=3.14159 effort=50.0 velocity=2.0; origin xyz=0 0 0 rpy=0 0 0 -> xyz=0.000000 -0.029745 0.071600 rpy=0 0 0; parent link_0 -> base_link
- joint joint_2: axis 0 0 1 -> 1 0 0; limit lower=0 upper=3.141592653589793 effort=1 velocity=1 -> lower=-3.14159 upper=3.14159 effort=50.0 velocity=2.0; origin xyz=0 0 0 rpy=0 0 0 -> xyz=0.008600 -0.010000 0.019250 rpy=0 0 0
- joint joint_3: axis 0 0 1 -> 1 0 0; limit lower=0 upper=3.141592653589793 effort=1 velocity=1 -> lower=-3.14159 upper=3.14159 effort=50.0 velocity=2.0; origin xyz=0 0 0 rpy=0 0 0 -> xyz=0.000000 0.000000 0.110490 rpy=0 0 0
- joint joint_4: axis 0 0 1 -> 1 0 0; limit lower=0 upper=3.141592653589793 effort=1 velocity=1 -> lower=-3.14159 upper=3.14159 effort=50.0 velocity=2.0; origin xyz=0 0 0 rpy=0 0 0 -> xyz=0.000000 -0.130491 0.000000 rpy=0 0 0
- joint joint_5: axis 0 0 1 -> 0 1 0; limit lower=0 upper=3.141592653589793 effort=1 velocity=1 -> lower=-3.14159 upper=3.14159 effort=50.0 velocity=2.0; origin xyz=0 0 0 rpy=0 0 0 -> xyz=0.010001 -0.067246 -0.000001 rpy=0 0 0

Commit message: restructure

File: ARM_control/models/robot.urdf (robot description, URDF)
Before this commit: robot robot_arm, 7 links, 6 joints
Joints:
- joint tool0_fixed: origin xyz=0 0 0 rpy=0 0 0 -> xyz=0.009849 -0.0687135 0 rpy=0 0 0
